Commit message: fixed bumper and added it to the simulater adapter

File: neato_robot/neato_description/urdf/neato_gazebo.urdf.xacro (robot description, xacro)
@@ -58,8 +58,8 @@
       <sensor type="contact" name="bumpers">
         <always_on>1</always_on>
-        <update_rate>50.0</update_rate>
+        <update_rate>10.0</update_rate>
         <visualize>true</visualize>
         <contact>
-          <collision>base_footprint_collision_base_link</collision>
+          <collision>base_footprint_fixed_joint_lump__base_link_collision_1</collision>
         </contact>
         <plugin name="gazebo_ros_bumper_controller" filename="libgazebo_ros_bumper.so">
