Commit message: added camera

File: neato_robot/neato_description/urdf/neato.urdf.xacro (robot description, xacro)
@@ -11,4 +11,5 @@
   <!-- neato -->
   <xacro:macro name="neato">
+	  <xacro:property name="camera_link" value="0.05" />
     <link name="base_footprint"/>
     <joint name="base_joint" type="fixed">
@@ -237,4 +238,31 @@
       </inertial>
     </link>
+  <joint name="camera_joint" type="fixed">
+    <axis xyz="0 1 0" />
+    <origin xyz="-0.1 0 0.25" rpy="0 0 0"/>
+    <parent link="base_link"/>
+    <child link="camera_link"/>
+  </joint>
+  <!-- Camera -->
+  <link name="camera_link">
+    <collision>
+      <origin xyz="0 0 0" rpy="0 0 0"/>
+      <geometry>
+    <box size="${camera_link} ${camera_link} ${camera_link}"/>
+      </geometry>
+    </collision>
+    <visual>
+      <origin xyz="0 0 0" rpy="0 0 0"/>
+      <geometry>
+    <box size="${camera_link} ${camera_link} ${camera_link}"/>
+      </geometry>
+      <material name="red"/>
+    </visual>
+    <inertial>
+      <mass value="1e-5" />
+      <origin xyz="0 0 0" rpy="0 0 0"/>
+      <inertia ixx="1e-6" ixy="0" ixz="0" iyy="1e-6" iyz="0" izz="1e-6" />
+    </inertial>
+  </link>
     <neato_sim/>
   </xacro:macro>

File: neato_robot/neato_description/urdf/neato_gazebo.urdf.xacro (robot description, xacro)
@@ -136,4 +136,44 @@
       </plugin>
       </gazebo>
+  <!-- camera -->
+  <gazebo reference="camera_link">
+    <sensor type="camera" name="camera">
+      <update_rate>30.0</update_rate>
+      <camera name="camera">
+        <horizontal_fov>1.3962634</horizontal_fov>
+        <image>
+          <width>800</width>
+          <height>800</height>
+          <format>R8G8B8</format>
+        </image>
+        <clip>
+          <near>0.02</near>
+          <far>300</far>
+        </clip>
+        <noise>
+          <type>gaussian</type>
+          <!-- Noise is sampled independently per pixel on each frame.
+               That pixel's noise value is added to each of its color
+               channels, which at that point lie in the range [0,1]. -->
+          <mean>0.0</mean>
+          <stddev>0.007</stddev>
+        </noise>
+      </camera>
+      <plugin name="camera_controller" filename="libgazebo_ros_camera.so">
+        <alwaysOn>true</alwaysOn>
+        <updateRate>0.0</updateRate>
+        <cameraName>camera</cameraName>
+        <imageTopicName>image_raw</imageTopicName>
+        <cameraInfoTopicName>camera_info</cameraInfoTopicName>
+        <frameName>camera_link</frameName>
+        <hackBaseline>0.07</hackBaseline>
+        <distortionK1>0.0</distortionK1>
+        <distortionK2>0.0</distortionK2>
+        <distortionK3>0.0</distortionK3>
+        <distortionT1>0.0</distortionT1>
+        <distortionT2>0.0</distortionT2>
+      </plugin>
+    </sensor>
+  </gazebo>
   </xacro:macro>
 </robot>

Commit message: reduce camera resolution.  move laser sensor up to avoid self collisiosn

File: neato_robot/neato_description/urdf/neato.urdf.xacro (robot description, xacro)
@@ -225,5 +225,7 @@
     </link>
     <joint name="laser_joint" type="fixed">
-      <origin xyz="-0.084 0 0.066" rpy="0 0 ${M_PI}" />
+      <!-- Using a higher z origin than the physical robot due to erroneous self-collisions of
+	   laser with the body of the robot (as determined by the ROS Gazebo plugin) -->
+      <origin xyz="-0.084 0 0.166" rpy="0 0 ${M_PI}" />
       <parent link="base_link"/>
       <child link="laser_link" />

File: neato_robot/neato_description/urdf/neato_gazebo.urdf.xacro (robot description, xacro)
@@ -90,5 +90,5 @@
         <plugin name="gazebo_ros_laser_controller" filename="libgazebo_ros_laser.so">
           <topicName>scan</topicName>
-          <frameName>laser_link</frameName>
+	  <frameName>laser_link</frameName>
         </plugin>
       </sensor>
@@ -143,6 +143,6 @@
         <horizontal_fov>1.3962634</horizontal_fov>
         <image>
-          <width>800</width>
-          <height>800</height>
+          <width>640</width>
+          <height>480</height>
           <format>R8G8B8</format>
         </image>

Commit message: testing light sources

File: neato_robot/neato_description/urdf/neato.urdf.xacro (robot description, xacro)
@@ -267,4 +267,22 @@
     </inertial>
   </link>
+      <link name='light_cylinder'>
+        <collision name='collision'>
+          <geometry>
+		  <cylinder radius="0.05" length="0.1"/>
+          </geometry>
+        </collision>
+        <visual name='visual'>
+          <geometry>
+		  <cylinder radius="0.05" length="0.1"/>
+          </geometry>
+        </visual>
+      </link>
+  <joint name="camera_to_light" type="fixed">
+    <axis xyz="0 1 0" />
+    <origin xyz="-0.1 0 0.25" rpy="0 0 0"/>
+    <parent link="camera_link"/>
+    <child link="light_cylinder"/>
+  </joint>
 </xacro:if>
     <xacro:neato_sim/>

File: neato_robot/neato_description/urdf/neato_gazebo.urdf.xacro (robot description, xacro)
@@ -199,5 +199,51 @@
       </plugin>
     </sensor>
-  </gazebo>
+    </gazebo>
+    <gazebo reference="light_cylinder">
+        <light name='light_source1' type='spot'>
+          <pose frame=''>0.25 0 0.25 0 -0.7854 0</pose>
+          <attenuation>
+            <range>30</range>
+            <linear>0.05</linear>
+          </attenuation>
+          <diffuse>1 0 0 1</diffuse>
+          <specular>1 0 0 1</specular>
+          <spot>
+            <inner_angle>0.3</inner_angle>
+            <outer_angle>0.35</outer_angle>
+            <falloff>1</falloff>
+          </spot>
+          <direction>0 0 -1</direction>
+        </light>
+        <light name='light_source2' type='spot'>
+          <pose frame=''>-0.25 0 0.25 0 0.7854 0</pose>
+          <attenuation>
+            <range>30</range>
+            <linear>0.05</linear>
+          </attenuation>
+          <diffuse>0 1 0 1</diffuse>
+          <specular>0 1 0 1</specular>
+          <spot>
+            <inner_angle>0.3</inner_angle>
+            <outer_angle>0.35</outer_angle>
+            <falloff>1</falloff>
+          </spot>
+          <direction>0 0 -1</direction>
+        </light>
+      <plugin name='light_control' filename='libFlashLightPlugin.so'>
+        <enable>true</enable>
+        <light>
+		<id>light_cylinder/light_source1</id>
+          <duration>0.1</duration>
+          <interval>0.4</interval>
+        </light>
+        <light>
+		<id>light_cylinder/light_source2</id>
+          <duration>0.05</duration>
+          <interval>0.05</interval>
+          <color>0.5 1 0.8</color>
+        </light>
+      </plugin>
+    </gazebo>
 </xacro:if>
   </xacro:macro>
