Commit message: customize shape from command line

File: com_workshop/urdf/blueCylinder.xacro (robot description, xacro)
@@ -2,4 +2,4 @@
 <robot xmlns:xacro="http://ros.org/wiki/xacro" name="blueCylinder">
 	<xacro:include filename="$(find com_workshop)/urdf/comShapes.xacro" />
-<xacro:blue_cylinder name="base_link" mass="5" radius=".42" length=".05"/>
+<xacro:blue_cylinder/>
 </robot>

File: com_workshop/urdf/comShapes.xacro (robot description, xacro)
@@ -1,48 +1,54 @@
 <?xml version="1.0"?>
 <robot xmlns:xacro="http://ros.org/wiki/xacro" name="testshape">
-<xacro:macro name="blue_cylinder" params="name mass radius length">
-    <link name="${name}">
+<xacro:macro name="blue_cylinder">
+     <xacro:arg name="radius" default="0.5" />
+     <xacro:arg name="mass" default="5" />
+     <xacro:arg name="length" default="1" />
+	<link name="base_link">
         <visual>
             <geometry>
-		    <cylinder length="${length}" radius="${radius}"/>
+		    <cylinder length="$(arg length)" radius="$(arg radius)"/>
             </geometry>
         </visual>
         <collision>
             <geometry>
-		    <cylinder length="${length}" radius="${radius}"/>
+		    <cylinder length="$(arg length)" radius="$(arg radius)"/>
             </geometry>
     </collision>
     <inertial>
-	    <mass value="${mass}" />
+	    <mass value="$(arg mass)" />
 	    <!-- http://scienceworld.wolfram.com/physics/MomentofInertiaCylinder.html -->
-	    <inertia ixx="${1/12*mass*length*length + 1/4*mass*radius*radius}" ixy="0.0" ixz="0.0" iyy="${1/12*mass*length*length + 1/4*mass*radius*radius}" iyz="0.0" izz="${1/2*mass*radius*radius}" />
+	    <inertia ixx="${1/12*$(arg mass)*$(arg length)*$(arg length) + 1/4*$(arg mass)*$(arg radius)*$(arg radius)}" ixy="0.0" ixz="0.0" iyy="${1/12*$(arg mass)*$(arg length)*$(arg length) + 1/4*$(arg mass)*$(arg radius)*$(arg radius)}" iyz="0.0" izz="${1/2*$(arg mass)*$(arg radius)*$(arg radius)}" />
     </inertial>
     </link>
-    <gazebo reference="${name}">
+    <gazebo reference="base_link">
    <material>Gazebo/Blue</material>
  </gazebo>
 </xacro:macro>
-<xacro:macro name="red_box" params="name mass length width height">
-    <link name="${name}">
+<xacro:macro name="red_box">
+     <xacro:arg name="mass" default="5" />
+     <xacro:arg name="length" default="1" />
+     <xacro:arg name="width" default="1" />
+     <xacro:arg name="height" default="1" />
+    <link name="base_link">
         <visual>
             <geometry>
-		    <box size="${length} ${width} ${height}"/>
+		    <box size="$(arg length) $(arg width) $(arg height)"/>
             </geometry>
         </visual>
         <collision>
             <geometry>
-		    <box size="${length} ${width} ${height}"/>
+		    <box size="$(arg length) $(arg width) $(arg height)"/>
             </geometry>
     </collision>
     <inertial>
-	    <mass value="${mass}" />
+	    <mass value="$(arg mass)" />
 	    <!-- https://en.wikipedia.org/wiki/List_of_moments_of_inertia#List_of_3D_inertia_tensors  Note: we are using length, width, height where they use width, height, depth -->
-	    <inertia ixx="${1/12*mass*(height*height + width*width)}" ixy="0.0" ixz="0.0" iyy="${1/12*mass*(height*height + length*length)}" iyz="0.0" izz="${1/12*mass*(length*length + width*width)}" />
+	    <inertia ixx="${1/12*$(arg mass)*($(arg height)*$(arg height) + $(arg width)*$(arg width))}" ixy="0.0" ixz="0.0" iyy="${1/12*$(arg mass)*($(arg height)*$(arg height) + $(arg length)*$(arg length))}" iyz="0.0" izz="${1/12*$(arg mass)*($(arg length)*$(arg length) + $(arg width)*$(arg width))}" />
     </inertial>
     </link>
-    <gazebo reference="${name}">
+    <gazebo reference="base_link">
    <material>Gazebo/Red</material>
  </gazebo>
 </xacro:macro>
-<!--<xacro:red_box name="base_link" mass="5" length=".42" width=".05" height="2"/>-->
 </robot>

File: com_workshop/urdf/redBox.xacro (robot description, xacro)
@@ -2,4 +2,4 @@
 <robot xmlns:xacro="http://ros.org/wiki/xacro" name="redBox">
 	<xacro:include filename="$(find com_workshop)/urdf/comShapes.xacro" />
-<xacro:red_box name="base_link" mass="5" length=".42" width=".05" height="2"/>
+<xacro:red_box/>
 </robot>

Commit message: changed xacros to be more flexible

File: com_workshop/urdf/blueCylinder.xacro (robot description, xacro)
@@ -1,5 +1,8 @@
 <?xml version="1.0"?>
 <robot xmlns:xacro="http://ros.org/wiki/xacro" name="blueCylinder">
+     <xacro:arg name="radius" default="0.5" />
+     <xacro:arg name="mass" default="5" />
+     <xacro:arg name="length" default="1" />
 	<xacro:include filename="$(find com_workshop)/urdf/comShapes.xacro" />
-<xacro:blue_cylinder/>
+<xacro:blue_cylinder radius="$(arg radius)" mass="$(arg mass)" length="$(arg length)"/>
 </robot>

File: com_workshop/urdf/comShapes.xacro (robot description, xacro)
@@ -1,23 +1,20 @@
 <?xml version="1.0"?>
 <robot xmlns:xacro="http://ros.org/wiki/xacro" name="testshape">
-<xacro:macro name="blue_cylinder">
-     <xacro:arg name="radius" default="0.5" />
-     <xacro:arg name="mass" default="5" />
-     <xacro:arg name="length" default="1" />
+<xacro:macro name="blue_cylinder" params="radius mass length">
 	<link name="base_link">
         <visual>
             <geometry>
-		    <cylinder length="$(arg length)" radius="$(arg radius)"/>
+		    <cylinder length="${length}" radius="${radius}"/>
             </geometry>
         </visual>
         <collision>
             <geometry>
-		    <cylinder length="$(arg length)" radius="$(arg radius)"/>
+		    <cylinder length="${length}" radius="${radius}"/>
             </geometry>
     </collision>
     <inertial>
-	    <mass value="$(arg mass)" />
+	    <mass value="{mass}" />
 	    <!-- http://scienceworld.wolfram.com/physics/MomentofInertiaCylinder.html -->
-	    <inertia ixx="${1/12*$(arg mass)*$(arg length)*$(arg length) + 1/4*$(arg mass)*$(arg radius)*$(arg radius)}" ixy="0.0" ixz="0.0" iyy="${1/12*$(arg mass)*$(arg length)*$(arg length) + 1/4*$(arg mass)*$(arg radius)*$(arg radius)}" iyz="0.0" izz="${1/2*$(arg mass)*$(arg radius)*$(arg radius)}" />
+	    <inertia ixx="${1/12*mass*length*length + 1/4*mass*radius*radius}" ixy="0.0" ixz="0.0" iyy="${1/12*mass*length*length + 1/4*mass*radius*radius}" iyz="0.0" izz="${1/2*mass*radius*radius}" />
     </inertial>
     </link>
@@ -26,24 +23,20 @@
  </gazebo>
 </xacro:macro>
-<xacro:macro name="red_box">
-     <xacro:arg name="mass" default="5" />
-     <xacro:arg name="length" default="1" />
-     <xacro:arg name="width" default="1" />
-     <xacro:arg name="height" default="1" />
+<xacro:macro name="red_box" params="mass length width height">
     <link name="base_link">
         <visual>
             <geometry>
-		    <box size="$(arg length) $(arg width) $(arg height)"/>
+		    <box size="${length} ${width} ${height}"/>
             </geometry>
         </visual>
         <collision>
             <geometry>
-		    <box size="$(arg length) $(arg width) $(arg height)"/>
+		    <box size="${length} ${width} ${height}"/>
             </geometry>
     </collision>
     <inertial>
-	    <mass value="$(arg mass)" />
+	    <mass value="${mass}" />
 	    <!-- https://en.wikipedia.org/wiki/List_of_moments_of_inertia#List_of_3D_inertia_tensors  Note: we are using length, width, height where they use width, height, depth -->
-	    <inertia ixx="${1/12*$(arg mass)*($(arg height)*$(arg height) + $(arg width)*$(arg width))}" ixy="0.0" ixz="0.0" iyy="${1/12*$(arg mass)*($(arg height)*$(arg height) + $(arg length)*$(arg length))}" iyz="0.0" izz="${1/12*$(arg mass)*($(arg length)*$(arg length) + $(arg width)*$(arg width))}" />
+	    <inertia ixx="${1/12*mass*(height*height + width*width)}" ixy="0.0" ixz="0.0" iyy="${1/12*mass*(height*height + length*length)}" iyz="0.0" izz="${1/12*mass*(length*length + width*width)}" />
     </inertial>
     </link>

File: com_workshop/urdf/redBox.xacro (robot description, xacro)
@@ -1,5 +1,9 @@
 <?xml version="1.0"?>
 <robot xmlns:xacro="http://ros.org/wiki/xacro" name="redBox">
+     <xacro:arg name="mass" default="5" />
+     <xacro:arg name="length" default="1" />
+     <xacro:arg name="width" default="1" />
+     <xacro:arg name="height" default="1" />
 	<xacro:include filename="$(find com_workshop)/urdf/comShapes.xacro" />
-<xacro:red_box/>
+<xacro:red_box mass="$(arg mass)" length="$(arg length)" width="$(arg width)" height="$(arg height)"/>
 </robot>

Commit message: allow for compound objects

File: com_workshop/urdf/blueCylinder.xacro (robot description, xacro)
@@ -1,8 +1,9 @@
 <?xml version="1.0"?>
 <robot xmlns:xacro="http://ros.org/wiki/xacro" name="blueCylinder">
+     <xacro:arg name="name" default="base_link" />
      <xacro:arg name="radius" default="0.5" />
      <xacro:arg name="mass" default="5" />
      <xacro:arg name="length" default="1" />
 	<xacro:include filename="$(find com_workshop)/urdf/comShapes.xacro" />
-<xacro:blue_cylinder radius="$(arg radius)" mass="$(arg mass)" length="$(arg length)"/>
+	<xacro:blue_cylinder name="$(arg name)" radius="$(arg radius)" mass="$(arg mass)" length="$(arg length)"/>
 </robot>

File: com_workshop/urdf/comShapes.xacro (robot description, xacro)
@@ -1,7 +1,8 @@
 <?xml version="1.0"?>
 <robot xmlns:xacro="http://ros.org/wiki/xacro" name="testshape">
-<xacro:macro name="blue_cylinder" params="radius mass length">
-	<link name="base_link">
+<xacro:macro name="blue_cylinder" params="name radius mass length x:=0 y:=0 z:=0">
+	<link name="${name}">
         <visual>
+	    <origin xyz="${x} ${y} ${z}"/>
             <geometry>
 		    <cylinder length="${length}" radius="${radius}"/>
@@ -9,4 +10,5 @@
         </visual>
         <collision>
+	    <origin xyz="${x} ${y} ${z}"/>
             <geometry>
 		    <cylinder length="${length}" radius="${radius}"/>
@@ -14,4 +16,5 @@
     </collision>
     <inertial>
+	    <origin xyz="${x} ${y} ${z}"/>
 	    <mass value="${mass}" />
 	    <!-- http://scienceworld.wolfram.com/physics/MomentofInertiaCylinder.html -->
@@ -19,16 +22,18 @@
     </inertial>
     </link>
-    <gazebo reference="base_link">
+    <gazebo reference="${name}">
    <material>Gazebo/Blue</material>
  </gazebo>
 </xacro:macro>
-<xacro:macro name="red_box" params="mass length width height">
-    <link name="base_link">
+<xacro:macro name="red_box" params="name mass length width height x:=0 y:=0 z:=0">
+    <link name="${name}">
         <visual>
-            <geometry>
+		<origin xyz="${x} ${y} ${z}"/>
+		<geometry>
 		    <box size="${length} ${width} ${height}"/>
             </geometry>
         </visual>
         <collision>
+	    <origin xyz="${x} ${y} ${z}"/>
             <geometry>
 		    <box size="${length} ${width} ${height}"/>
@@ -41,5 +46,5 @@
     </inertial>
     </link>
-    <gazebo reference="base_link">
+    <gazebo reference="${name}">
    <material>Gazebo/Red</material>
  </gazebo>

File: com_workshop/urdf/redBox.xacro (robot description, xacro)
@@ -1,4 +1,5 @@
 <?xml version="1.0"?>
 <robot xmlns:xacro="http://ros.org/wiki/xacro" name="redBox">
+     <xacro:arg name="name" default="base_link" />
      <xacro:arg name="mass" default="5" />
      <xacro:arg name="length" default="1" />
@@ -6,4 +7,4 @@
      <xacro:arg name="height" default="1" />
 	<xacro:include filename="$(find com_workshop)/urdf/comShapes.xacro" />
-<xacro:red_box mass="$(arg mass)" length="$(arg length)" width="$(arg width)" height="$(arg height)"/>
+<xacro:red_box name="$(arg name)" mass="$(arg mass)" length="$(arg length)" width="$(arg width)" height="$(arg height)"/>
 </robot>
