Commit message: fixed typo

File: com_workshop/urdf/comShapes.xacro (robot description, xacro)
@@ -14,5 +14,5 @@
     </collision>
     <inertial>
-	    <mass value="{mass}" />
+	    <mass value="${mass}" />
 	    <!-- http://scienceworld.wolfram.com/physics/MomentofInertiaCylinder.html -->
 	    <inertia ixx="${1/12*mass*length*length + 1/4*mass*radius*radius}" ixy="0.0" ixz="0.0" iyy="${1/12*mass*length*length + 1/4*mass*radius*radius}" iyz="0.0" izz="${1/2*mass*radius*radius}" />

Commit message: more flexible... able to build compound objects

File: com_workshop/urdf/comShapes.xacro (robot description, xacro)
@@ -1,8 +1,8 @@
 <?xml version="1.0"?>
 <robot xmlns:xacro="http://ros.org/wiki/xacro" name="testshape">
-<xacro:macro name="blue_cylinder" params="name radius mass length x:=0 y:=0 z:=0">
+<xacro:macro name="blue_cylinder" params="name radius mass length">
 	<link name="${name}">
         <visual>
-	    <origin xyz="${x} ${y} ${z}"/>
+	    <origin xyz="0 0 ${length/2}"/>
             <geometry>
 		    <cylinder length="${length}" radius="${radius}"/>
@@ -10,5 +10,5 @@
         </visual>
         <collision>
-	    <origin xyz="${x} ${y} ${z}"/>
+	    <origin xyz="0 0 ${length/2}"/>
             <geometry>
 		    <cylinder length="${length}" radius="${radius}"/>
@@ -16,5 +16,5 @@
     </collision>
     <inertial>
-	    <origin xyz="${x} ${y} ${z}"/>
+	    <origin xyz="0 0 ${length/2}"/>
 	    <mass value="${mass}" />
 	    <!-- http://scienceworld.wolfram.com/physics/MomentofInertiaCylinder.html -->
@@ -26,8 +26,8 @@
  </gazebo>
 </xacro:macro>
-<xacro:macro name="red_box" params="name mass length width height x:=0 y:=0 z:=0">
+<xacro:macro name="red_box" params="name mass length width height">
     <link name="${name}">
         <visual>
-		<origin xyz="${x} ${y} ${z}"/>
+		<origin xyz="0 0 ${height/2}"/>
 		<geometry>
 		    <box size="${length} ${width} ${height}"/>
@@ -35,5 +35,5 @@
         </visual>
         <collision>
-	    <origin xyz="${x} ${y} ${z}"/>
+	    <origin xyz="0 0 ${height/2}"/>
             <geometry>
 		    <box size="${length} ${width} ${height}"/>
@@ -41,4 +41,5 @@
     </collision>
     <inertial>
+	    <origin xyz="0 0 ${height/2}"/>
 	    <mass value="${mass}" />
 	    <!-- https://en.wikipedia.org/wiki/List_of_moments_of_inertia#List_of_3D_inertia_tensors  Note: we are using length, width, height where they use width, height, depth -->
